File: ethernet-sniffer/7seg-display.sch (KiCad schematic (older format))
At the start: 11 parts, among them Q201 2N3904, Q202 2N3904

Commit message: Add files via upload
Parts:
- Q201, Q202: footprint Package_TO_SOT_THT:TO-92_Inline -> Package_TO_SOT_SMD:SOT-23
Changed lines of the file:
@@
 F 0 "Q202" H 4841 3946 50  0000 L CNN
 F 1 "2N3904" H 4841 3855 50  0000 L CNN
-F 2 "Package_TO_SOT_THT:TO-92_Inline" H 4850 3825 50  0001 L CIN
+F 2 "Package_TO_SOT_SMD:SOT-23" H 4850 3825 50  0001 L CIN
 F 3 "https://www.fairchildsemi.com/datasheets/2N/2N3904.pdf" H 4650 3900 50  0001 L CNN
 	1    4650 3900
@@
 F 0 "Q201" H 4441 4446 50  0000 L CNN
 F 1 "2N3904" H 4441 4355 50  0000 L CNN
-F 2 "Package_TO_SOT_THT:TO-92_Inline" H 4450 4325 50  0001 L CIN
+F 2 "Package_TO_SOT_SMD:SOT-23" H 4450 4325 50  0001 L CIN
 F 3 "https://www.fairchildsemi.com/datasheets/2N/2N3904.pdf" H 4250 4400 50  0001 L CNN
 	1    4250 4400
