File: ethernet-sniffer/7segment.sch (KiCad schematic (older format))
At the start: 7 parts

Commit message: Add files via upload
Added again in the right folder this time hopefully
Changed lines of the file:
@@
 AR Path="/604ADF19/604B8E8A/5F24E765" Ref="D303"  Part="1"
 AR Path="/604ADF19/604B8EA0/5F24E765" Ref="D403"  Part="1"
-F 0 "D303" H 5000 2535 50  0000 C CNN
+F 0 "D403" H 5000 2535 50  0000 C CNN
 F 1 "A" H 5000 2444 50  0000 C CNN
 F 2 "LED_SMD:LED_0402_1005Metric" V 5000 2300 50  0001 C CNN
@@
 AR Path="/604ADF19/604B8E8A/5F24E76B" Ref="D301"  Part="1"
 AR Path="/604ADF19/604B8EA0/5F24E76B" Ref="D401"  Part="1"
-F 0 "D301" V 4550 2550 50  0000 L CNN
+F 0 "D401" V 4550 2550 50  0000 L CNN
 F 1 "B" V 4650 2600 50  0000 L CNN
 F 2 "LED_SMD:LED_0402_1005Metric" V 4600 2750 50  0001 C CNN
@@
 AR Path="/604ADF19/604B8E8A/5F24E771" Ref="D302"  Part="1"
 AR Path="/604ADF19/604B8EA0/5F24E771" Ref="D402"  Part="1"
-F 0 "D302" V 4646 3582 50  0000 R CNN
+F 0 "D402" V 4646 3582 50  0000 R CNN
 F 1 "C" V 4555 3582 50  0000 R CNN
 F 2 "LED_SMD:LED_0402_1005Metric" V 4600 3650 50  0001 C CNN
@@
 AR Path="/604ADF19/604B8E8A/5F24E777" Ref="D305"  Part="1"
 AR Path="/604ADF19/604B8EA0/5F24E777" Ref="D405"  Part="1"
-F 0 "D305" H 5000 4335 50  0000 C CNN
+F 0 "D405" H 5000 4335 50  0000 C CNN
 F 1 "D" H 5000 4244 50  0000 C CNN
 F 2 "LED_SMD:LED_0402_1005Metric" V 5000 4100 50  0001 C CNN
@@
 AR Path="/604ADF19/604B8E8A/5F24E77D" Ref="D307"  Part="1"
 AR Path="/604ADF19/604B8EA0/5F24E77D" Ref="D407"  Part="1"
-F 0 "D307" V 5450 3850 50  0000 R CNN
+F 0 "D407" V 5450 3850 50  0000 R CNN
 F 1 "E" V 5350 3800 50  0000 R CNN
 F 2 "LED_SMD:LED_0402_1005Metric" V 5400 3650 50  0001 C CNN
@@
 AR Path="/604ADF19/604B8E8A/5F24E783" Ref="D306"  Part="1"
 AR Path="/604ADF19/604B8EA0/5F24E783" Ref="D406"  Part="1"
-F 0 "D306" V 5446 2682 50  0000 R CNN
+F 0 "D406" V 5446 2682 50  0000 R CNN
 F 1 "F" V 5355 2682 50  0000 R CNN
 F 2 "LED_SMD:LED_0402_1005Metric" V 5400 2750 50  0001 C CNN
@@
 AR Path="/604ADF19/604B8E8A/5F24E789" Ref="D304"  Part="1"
 AR Path="/604ADF19/604B8EA0/5F24E789" Ref="D404"  Part="1"
-F 0 "D304" H 5000 3435 50  0000 C CNN
+F 0 "D404" H 5000 3435 50  0000 C CNN
 F 1 "G" H 5000 3344 50  0000 C CNN
 F 2 "LED_SMD:LED_0402_1005Metric" V 5000 3200 50  0001 C CNN

Commit message: Add files via upload
Parts:
- D301, D302, D303, D304, D305, D306, D307: footprint LED_SMD:LED_0402_1005Metric -> LED_SMD:LED_0603_1608Metric
Changed lines of the file:
@@
 F 0 "D403" H 5000 2535 50  0000 C CNN
 F 1 "A" H 5000 2444 50  0000 C CNN
-F 2 "LED_SMD:LED_0402_1005Metric" V 5000 2300 50  0001 C CNN
+F 2 "LED_SMD:LED_0603_1608Metric" V 5000 2300 50  0001 C CNN
 F 3 "~" V 5000 2300 50  0001 C CNN
 	1    5000 2300
@@
 F 0 "D401" V 4550 2550 50  0000 L CNN
 F 1 "B" V 4650 2600 50  0000 L CNN
-F 2 "LED_SMD:LED_0402_1005Metric" V 4600 2750 50  0001 C CNN
+F 2 "LED_SMD:LED_0603_1608Metric" V 4600 2750 50  0001 C CNN
 F 3 "~" V 4600 2750 50  0001 C CNN
 	1    4600 2750
@@
 F 0 "D402" V 4646 3582 50  0000 R CNN
 F 1 "C" V 4555 3582 50  0000 R CNN
-F 2 "LED_SMD:LED_0402_1005Metric" V 4600 3650 50  0001 C CNN
+F 2 "LED_SMD:LED_0603_1608Metric" V 4600 3650 50  0001 C CNN
 F 3 "~" V 4600 3650 50  0001 C CNN
 	1    4600 3650
@@
 F 0 "D405" H 5000 4335 50  0000 C CNN
 F 1 "D" H 5000 4244 50  0000 C CNN
-F 2 "LED_SMD:LED_0402_1005Metric" V 5000 4100 50  0001 C CNN
+F 2 "LED_SMD:LED_0603_1608Metric" V 5000 4100 50  0001 C CNN
 F 3 "~" V 5000 4100 50  0001 C CNN
 	1    5000 4100
@@
 F 0 "D407" V 5450 3850 50  0000 R CNN
 F 1 "E" V 5350 3800 50  0000 R CNN
-F 2 "LED_SMD:LED_0402_1005Metric" V 5400 3650 50  0001 C CNN
+F 2 "LED_SMD:LED_0603_1608Metric" V 5400 3650 50  0001 C CNN
 F 3 "~" V 5400 3650 50  0001 C CNN
 	1    5400 3650
@@
 F 0 "D406" V 5446 2682 50  0000 R CNN
 F 1 "F" V 5355 2682 50  0000 R CNN
-F 2 "LED_SMD:LED_0402_1005Metric" V 5400 2750 50  0001 C CNN
+F 2 "LED_SMD:LED_0603_1608Metric" V 5400 2750 50  0001 C CNN
 F 3 "~" V 5400 2750 50  0001 C CNN
 	1    5400 2750
@@
 F 0 "D404" H 5000 3435 50  0000 C CNN
 F 1 "G" H 5000 3344 50  0000 C CNN
-F 2 "LED_SMD:LED_0402_1005Metric" V 5000 3200 50  0001 C CNN
+F 2 "LED_SMD:LED_0603_1608Metric" V 5000 3200 50  0001 C CNN
 F 3 "~" V 5000 3200 50  0001 C CNN
 	1    5000 3200
