File: ethernet-sniffer/FPGA.sch (KiCad schematic (older format))
At the start: 82 parts, among them J701 JTAG, SW701 RESET, U701 LM317_3PinPackage, U702 AMS1117-3.3, U703 AMS1117-3.3, U704 AMS1117-3.3, U705 AMS1117-3.3, U706 AMS1117-3.3, U707 XC6SLX9-TQG144

Commit message: Add files via upload
Parts:
- removed C707, C708, C709, C710: 100u, Capacitor_SMD:C_0603_1608Metric, symbol Device:C_Small
- removed C719, C720, C721, C722: 10u, Capacitor_SMD:C_0402_1005Metric, symbol Device:C_Small
- removed C727, C728, C729, C730: 100n, Capacitor_SMD:C_0402_1005Metric, symbol Device:C_Small
- removed C731: 4u7, Capacitor_SMD:C_0402_1005Metric, symbol Device:C_Small
- removed C735, C736, C737, C738: 10n, Capacitor_SMD:C_0402_1005Metric, symbol Device:C_Small
- removed C739, C742: 470n, Capacitor_SMD:C_0402_1005Metric, symbol Device:C_Small
- removed D702, D703, D704, D705: LED_Small, LED_SMD:LED_0402_1005Metric, symbol Device:LED_Small
- removed R705, R706, R707, R708: 200, Resistor_SMD:R_0402_1005Metric, symbol Device:R_Small_US
- removed R709, R710, R711, R712: 0, Resistor_SMD:R_0402_1005Metric, symbol Device:R_Small_US
- removed TP703, TP704, TP705, TP706: TP 3.3V VCCAUX, TestPoint:TestPoint_Keystone_5015_Micro-Minature, symbol Connector:TestPoint
- removed U703, U704, U705, U706: AMS1117-3.3, Package_TO_SOT_SMD:SOT-223-3_TabPin2, symbol Regulator_Linear:AMS1117-3.3
- added C1012: 100n, Capacitor_SMD:C_0402_1005Metric, symbol Device:C_Small
- added D707: INIT, LED_SMD:LED_0603_1608Metric, symbol Device:LED_Small
- added Q701: 2N3904, Package_TO_SOT_SMD:SOT-23, symbol Transistor_BJT:2N3904
- added R1141, R1142, R714, R717: 100, Resistor_SMD:R_0402_1005Metric, symbol Device:R_Small_US
- added R1143, R1144, R1145, R1146: 1k, Resistor_SMD:R_0402_1005Metric, symbol Device:R_Small_US
- added R1147, R1148, R719, R721, R722, R723: 2k2, Resistor_SMD:R_0402_1005Metric, symbol Device:R_Small_US
- added R715, R716, R720: 200, Resistor_SMD:R_0402_1005Metric, symbol Device:R_Small_US
- added R718: 10k, Resistor_SMD:R_0402_1005Metric, symbol Device:R_Small_US
- added U708: W25Q128JVS, Package_SO:SOIC-8_5.23x5.23mm_P1.27mm, symbol Memory_Flash:W25Q128JVS
- C701, C702, C704, C723, C732, C741, C743: value 4u7 -> 100n
- C703, C711, C716, C724, C740, C746, C747, C748: value 470n -> 100n
- C705, C706: value 100u -> 4u7; footprint Capacitor_SMD:C_0603_1608Metric -> Capacitor_SMD:C_0402_1005Metric
- C712, C713, C714, C715, C744, C745: value 4u7 -> 100n; footprint Capacitor_SMD:C_0603_1608Metric -> Capacitor_SMD:C_0402_1005Metric
- C725: value 1u -> 4u7
- C726: value 100n -> 4u7
- C733: value 100n -> 470n
- C734: value 10n -> 470n
- D701: footprint LED_SMD:LED_0402_1005Metric -> LED_SMD:LED_0603_1608Metric
- D706: value DONE -> INIT; footprint LED_SMD:LED_0402_1005Metric -> LED_SMD:LED_0603_1608Metric
- J701: footprint Connector_PinHeader_1.27mm:PinHeader_2x07_P1.27mm_Vertical -> Connector_PinHeader_2.54mm:PinHeader_2x07_P2.54mm_Vertical
Connections:
- net labels added: CCLK, CSO_B, DIN, DONE, INIT, INIT_B, M0, M1, MOSI, PHY1_CLK_GEN, PHY2_CLK_GEN, PHY3_CLK_GEN, PROGRAM, SPI_CLK, SPI_CS, SPI_MISO, SPI_MOSI, TCK, TDI, TDO, TMS, VCCO_3V3
- net labels removed: CLK_OUT, VCCAUX_3V3, VCCO_BANK0_3V3, VCCO_BANK1_3V3, VCCO_BANK2_3V3, VCCO_BANK3_3V3
- wire segments 351 -> 289
- no-connect marks 56 -> 19
Other:
- note added: "VCC 3.3V"
- note removed: "VCCAUX 3.3V"
- note removed: "VCCO BANK0 3.3V"
- note removed: "VCCO BANK1 3.3V"
- note removed: "VCCO BANK2 3.3V"
- note removed: "VCCO BANK3 3.3V"
- moved on the sheet: J701, SW701, U707C, U707D
