File: ethernet-sniffer/PHY.sch (KiCad schematic (older format))
At the start: 72 parts, among them J1002 SNI_MODE, J1003 PHY_AD1, J1004 PHY_AD2, J1005 PHY_AD3, J1006 PHY_AD4, J1007 MDIX_EN, J1008 Conn_01x03, J1009 PHY_AD0, J1010 ~RESET, J1011 POWER_DOWN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

Commit message: Add files via upload
Added again in the right folder this time hopefully
Parts:
- removed J1002: SNI_MODE, Connector_PinHeader_1.27mm:PinHeader_1x03_P1.27mm_Vertical, symbol Connector_Generic:Conn_01x03
- removed J1003: PHY_AD1, Connector_PinHeader_1.27mm:PinHeader_1x03_P1.27mm_Vertical, symbol Connector_Generic:Conn_01x03
- removed J1004: PHY_AD2, Connector_PinHeader_1.27mm:PinHeader_1x03_P1.27mm_Vertical, symbol Connector_Generic:Conn_01x03
- removed J1005: PHY_AD3, Connector_PinHeader_1.27mm:PinHeader_1x03_P1.27mm_Vertical, symbol Connector_Generic:Conn_01x03
- removed J1006: PHY_AD4, Connector_PinHeader_1.27mm:PinHeader_1x03_P1.27mm_Vertical, symbol Connector_Generic:Conn_01x03
- removed J1007: MDIX_EN, Connector_PinHeader_1.27mm:PinHeader_1x03_P1.27mm_Vertical, symbol Connector_Generic:Conn_01x03
- removed J1008, J1012: Conn_01x03, Connector_PinHeader_1.27mm:PinHeader_1x03_P1.27mm_Vertical, symbol Connector_Generic:Conn_01x03
- removed J1009: PHY_AD0, Connector_PinHeader_1.27mm:PinHeader_1x03_P1.27mm_Vertical, symbol Connector_Generic:Conn_01x03
- removed J1010: ~RESET, Connector_PinHeader_1.27mm:PinHeader_1x03_P1.27mm_Vertical, symbol Connector_Generic:Conn_01x03
- removed J1011: POWER_DOWN, Connector_PinHeader_1.27mm:PinHeader_1x03_P1.27mm_Vertical, symbol Connector_Generic:Conn_01x03
- removed J1013: AN0, Connector_PinHeader_1.27mm:PinHeader_1x03_P1.27mm_Vertical, symbol Connector_Generic:Conn_01x03
- removed J1014: AN1, Connector_PinHeader_1.27mm:PinHeader_1x03_P1.27mm_Vertical, symbol Connector_Generic:Conn_01x03
- removed J1015: AN_EN, Connector_PinHeader_1.27mm:PinHeader_1x03_P1.27mm_Vertical, symbol Connector_Generic:Conn_01x03
- added JP1001: SNI_MODE, Jumper:SolderJumper-3_P1.3mm_Open_RoundedPad1.0x1.5mm, symbol Device:Jumper_NC_Dual
- added JP1002: PHY_AD1, Jumper:SolderJumper-3_P1.3mm_Open_RoundedPad1.0x1.5mm, symbol Device:Jumper_NC_Dual
- added JP1003: PHY_AD2, Jumper:SolderJumper-3_P1.3mm_Open_RoundedPad1.0x1.5mm, symbol Device:Jumper_NC_Dual
- added JP1004: PHY_AD3, Jumper:SolderJumper-3_P1.3mm_Open_RoundedPad1.0x1.5mm, symbol Device:Jumper_NC_Dual
- added JP1005: PHY_AD4, Jumper:SolderJumper-3_P1.3mm_Open_RoundedPad1.0x1.5mm, symbol Device:Jumper_NC_Dual
- added JP1006: MDIX_EN, Jumper:SolderJumper-3_P1.3mm_Open_RoundedPad1.0x1.5mm, symbol Device:Jumper_NC_Dual
- added JP1007: MII_MODE, Jumper:SolderJumper-3_P1.3mm_Open_RoundedPad1.0x1.5mm, symbol Device:Jumper_NC_Dual
- added JP1008: PHY_AD0, Jumper:SolderJumper-3_P1.3mm_Open_RoundedPad1.0x1.5mm, symbol Device:Jumper_NC_Dual
- added JP1009: LED_CFG, Jumper:SolderJumper-3_P1.3mm_Open_RoundedPad1.0x1.5mm, symbol Device:Jumper_NC_Dual
- added JP1010: ~RESET, Jumper:SolderJumper-3_P1.3mm_Open_RoundedPad1.0x1.5mm, symbol Device:Jumper_NC_Dual
- added JP1011: POWER_DOWN, Jumper:SolderJumper-3_P1.3mm_Open_RoundedPad1.0x1.5mm, symbol Device:Jumper_NC_Dual
- added JP1012: AN0, Jumper:SolderJumper-3_P1.3mm_Open_RoundedPad1.0x1.5mm, symbol Device:Jumper_NC_Dual
- added JP1013: AN1, Jumper:SolderJumper-3_P1.3mm_Open_RoundedPad1.0x1.5mm, symbol Device:Jumper_NC_Dual
- added JP1014: AN_EN, Jumper:SolderJumper-3_P1.3mm_Open_RoundedPad1.0x1.5mm, symbol Device:Jumper_NC_Dual
Connections:
- net AN0: now also JP1012.2
- net AN1: now also JP1013.2
- net AN_EN: now also JP1014.2
- net CRS_DV: now also JP1009.2
- net MDIX_EN: now also JP1006.2
- net PHY_AD0: now also JP1008.2
- net PHY_AD3: now also JP1004.2
- net PHY_AD4: now also JP1005.2
- net POWER_DOWN: now also JP1011.2
- net RXD_0: now also JP1002.2
- net RXD_1: now also JP1003.2
- net RX_DV: now also JP1007.2
- net SNI_MODE: now also JP1001.2
- net ~RESET: now also JP1010.2
- net at R801.2: now also JP1001.1
- net at R802.1: now also JP1001.3
- net at R803.2: now also JP1002.1
- net at R804.1: now also JP1002.3
- net at R805.2: now also JP1003.1
- net at R806.1: now also JP1003.3
- net at R807.2: now also JP1004.1
- net at R808.1: now also JP1004.3
- net at R809.2: now also JP1005.1
- net at R810.1: now also JP1005.3
- net at R811.2: now also JP1006.1
- net at R812.1: now also JP1006.3
- net at R813.2: now also JP1007.1
- net at R814.1: now also JP1007.3
- net at R815.2: now also JP1008.1
- net at R816.1: now also JP1008.3
- net at R824.2: now also JP1009.1
- net at R825.1: now also JP1009.3
- net at R826.2: now also JP1010.1
- net at R827.1: now also JP1010.3
- net at R830.2: now also JP1011.1
- net at R831.1: now also JP1011.3
- net at R835.2: now also JP1012.1
- net at R836.1: now also JP1012.3
- net at R837.2: now also JP1013.1
- net at R838.1: now also JP1013.3
- net at R839.2: now also JP1014.1
- net at R840.1: now also JP1014.3
Other:
- moved on the sheet: R901, R902, R903, R904, R905, R906, R907, R908, R909, R910, R911, R912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

Commit message: Add files via upload
Parts:
- C801, C802, C808: footprint Capacitor_SMD:C_0603_1608Metric -> Capacitor_SMD:C_0402_1005Metric
- D801, D802, D803: footprint LED_SMD:LED_0402_1005Metric -> LED_SMD:LED_0603_1608Metric
