File: ethernet-sniffer/USBUART.sch (KiCad schematic (older format))
At the start: 7 parts, among them U501 CH340G, Y501 12MHz

Commit message: Add files via upload
Parts:
- Y501: footprint Crystal:Crystal_SMD_0603-2Pin_6.0x3.5mm_HandSoldering -> Crystal:Crystal_SMD_0603-2Pin_6.0x3.5mm
Changed lines of the file:
@@
 F 0 "Y501" V 2054 2938 50  0000 L CNN
 F 1 "12MHz" V 2145 2938 50  0000 L CNN
-F 2 "Crystal:Crystal_SMD_0603-2Pin_6.0x3.5mm_HandSoldering" H 2100 2850 50  0001 C CNN
+F 2 "Crystal:Crystal_SMD_0603-2Pin_6.0x3.5mm" H 2100 2850 50  0001 C CNN
 F 3 "~" H 2100 2850 50  0001 C CNN
 	1    2100 2850
