File: ethernet-sniffer/ethernet-sniffer.kicad_pcb (KiCad board)
At the start: 4 copper layers, 162.4 x 370.8 mm, 448 parts, among them J1001 RJMG1BD3B8K1ANR, J1002 SNI_MODE, J1003 PHY_AD1, J1004 PHY_AD2, J1005 PHY_AD3, J1006 PHY_AD4, J1007 MDIX_EN, J1008 Conn_01x03, J1009 PHY_AD0, J101 Conn_01x10, J1010 ~RESET, J1011 POWER_DOWN, J1012 Conn_01x03, J1013 AN0, J1014 AN1, J1015 AN_EN, J102 USB_B_Micro, J1101 RJMG1BD3B8K1ANR, J1102 SNI_MODE, J1103 PHY_AD1, J1104 PHY_AD2, J1105 PHY_AD3, J1106 PHY_AD4, J1107 MDIX_EN, J1108 Conn_01x03, J1109 PHY_AD0, J1110 ~RESET, J1111 POWER_DOWN, J1112 Conn_01x03, J1113 AN0, J1114 AN1, J1115 AN_EN, J601 Debug Header, J602 Extension Port A, J603 Extension Port B, J604 Extension Port E, J605 Extension Port C, J606 Extension Port D, J607 BOOT0, J608 BOOT1, J701 JTAG, J801 RJMG1BD3B8K1ANR, J802 SNI_MODE, J803 PHY_AD1, J804 PHY_AD2, J805 PHY_AD3, J806 PHY_AD4, J807 MDIX_EN, J808 Conn_01x03, J809 PHY_AD0, J810 ~RESET, J811 POWER_DOWN, J812 Conn_01x03, J813 AN0, J814 AN1, J815 AN_EN, J901 RJMG1BD3B8K1ANR, J902 SNI_MODE, J903 PHY_AD1, J904 PHY_AD2, J905 PHY_AD3, J906 PHY_AD4, J907 MDIX_EN, J908 Conn_01x03, J909 PHY_AD0, J910 ~RESET, J911 POWER_DOWN, J912 Conn_01x03, J913 AN0, J914 AN1, J915 AN_EN, Q201 2N3904, Q202 2N3904, SW601 SW_Push, SW701 RESET, U1001 AMS1117-3.3, U1002 DP83848C, U1101 AMS1117-3.3, U1102 DP83848C, U501 CH340G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

Commit message: Add files via upload
Added again in the right folder this time hopefully
Parts:
- removed J1002, J1102, J802, J902: SNI_MODE, Connector_PinHeader_1.27mm:PinHeader_1x03_P1.27mm_Vertical
- removed J1003, J1103, J803, J903: PHY_AD1, Connector_PinHeader_1.27mm:PinHeader_1x03_P1.27mm_Vertical
- removed J1004, J1104, J804, J904: PHY_AD2, Connector_PinHeader_1.27mm:PinHeader_1x03_P1.27mm_Vertical
- removed J1005, J1105, J805, J905: PHY_AD3, Connector_PinHeader_1.27mm:PinHeader_1x03_P1.27mm_Vertical
- removed J1006, J1106, J806, J906: PHY_AD4, Connector_PinHeader_1.27mm:PinHeader_1x03_P1.27mm_Vertical
- removed J1007, J1107, J807, J907: MDIX_EN, Connector_PinHeader_1.27mm:PinHeader_1x03_P1.27mm_Vertical
- removed J1008, J1012, J1108, J1112, J808, J812, J908, J912: Conn_01x03, Connector_PinHeader_1.27mm:PinHeader_1x03_P1.27mm_Vertical
- removed J1009, J1109, J809, J909: PHY_AD0, Connector_PinHeader_1.27mm:PinHeader_1x03_P1.27mm_Vertical
- removed J1010, J1110, J810, J910: ~RESET, Connector_PinHeader_1.27mm:PinHeader_1x03_P1.27mm_Vertical
- removed J1011, J1111, J811, J911: POWER_DOWN, Connector_PinHeader_1.27mm:PinHeader_1x03_P1.27mm_Vertical
- removed J1013, J1113, J813, J913: AN0, Connector_PinHeader_1.27mm:PinHeader_1x03_P1.27mm_Vertical
- removed J1014, J1114, J814, J914: AN1, Connector_PinHeader_1.27mm:PinHeader_1x03_P1.27mm_Vertical
- removed J1015, J1115, J815, J915: AN_EN, Connector_PinHeader_1.27mm:PinHeader_1x03_P1.27mm_Vertical
- added JP1001: SNI_MODE, Jumper:SolderJumper-3_P1.3mm_Open_RoundedPad1.0x1.5mm, B.Cu at (134.0, 50.4)
- added JP1002: PHY_AD1, Jumper:SolderJumper-3_P1.3mm_Open_RoundedPad1.0x1.5mm, B.Cu at (134.4, 57.0)
- added JP1003: PHY_AD2, Jumper:SolderJumper-3_P1.3mm_Open_RoundedPad1.0x1.5mm, B.Cu at (131.6, 57.0)
- added JP1004: PHY_AD3, Jumper:SolderJumper-3_P1.3mm_Open_RoundedPad1.0x1.5mm, B.Cu at (139.6, 50.4)
- added JP1005: PHY_AD4, Jumper:SolderJumper-3_P1.3mm_Open_RoundedPad1.0x1.5mm, B.Cu at (136.8, 50.4)
- added JP1006: MDIX_EN, Jumper:SolderJumper-3_P1.3mm_Open_RoundedPad1.0x1.5mm, B.Cu at (137.2, 63.8)
- added JP1007: MII_MODE, Jumper:SolderJumper-3_P1.3mm_Open_RoundedPad1.0x1.5mm, B.Cu at (131.6, 63.8)
- added JP1008: PHY_AD0, Jumper:SolderJumper-3_P1.3mm_Open_RoundedPad1.0x1.5mm, B.Cu at (137.2, 57.0)
- added JP1009: LED_CFG, Jumper:SolderJumper-3_P1.3mm_Open_RoundedPad1.0x1.5mm, B.Cu at (134.4, 63.8)
- added JP1010: ~RESET, Jumper:SolderJumper-3_P1.3mm_Open_RoundedPad1.0x1.5mm, B.Cu at (125.9, 70.9)
- added JP1011: POWER_DOWN, Jumper:SolderJumper-3_P1.3mm_Open_RoundedPad1.0x1.5mm, B.Cu at (131.2, 50.4)
- added JP1012: AN0, Jumper:SolderJumper-3_P1.3mm_Open_RoundedPad1.0x1.5mm, B.Cu at (125.9, 68.1)
- added JP1013: AN1, Jumper:SolderJumper-3_P1.3mm_Open_RoundedPad1.0x1.5mm, B.Cu at (120.7, 70.9)
- added JP1014: AN_EN, Jumper:SolderJumper-3_P1.3mm_Open_RoundedPad1.0x1.5mm, B.Cu at (115.6, 70.9)
- added JP1101: SNI_MODE, Jumper:SolderJumper-3_P1.3mm_Open_RoundedPad1.0x1.5mm, B.Cu at (134.6, 116.1)
- added JP1102: PHY_AD1, Jumper:SolderJumper-3_P1.3mm_Open_RoundedPad1.0x1.5mm, B.Cu at (135.0, 122.7)
- added JP1103: PHY_AD2, Jumper:SolderJumper-3_P1.3mm_Open_RoundedPad1.0x1.5mm, B.Cu at (132.2, 122.7)
- added JP1104: PHY_AD3, Jumper:SolderJumper-3_P1.3mm_Open_RoundedPad1.0x1.5mm, B.Cu at (140.2, 116.1)
- added JP1105: PHY_AD4, Jumper:SolderJumper-3_P1.3mm_Open_RoundedPad1.0x1.5mm, B.Cu at (137.4, 116.1)
- added JP1106: MDIX_EN, Jumper:SolderJumper-3_P1.3mm_Open_RoundedPad1.0x1.5mm, B.Cu at (137.8, 129.4)
- added JP1107: MII_MODE, Jumper:SolderJumper-3_P1.3mm_Open_RoundedPad1.0x1.5mm, B.Cu at (132.2, 129.4)
- added JP1108: PHY_AD0, Jumper:SolderJumper-3_P1.3mm_Open_RoundedPad1.0x1.5mm, B.Cu at (137.8, 122.7)
- added JP1109: LED_CFG, Jumper:SolderJumper-3_P1.3mm_Open_RoundedPad1.0x1.5mm, B.Cu at (135.0, 129.4)
- added JP1110: ~RESET, Jumper:SolderJumper-3_P1.3mm_Open_RoundedPad1.0x1.5mm, B.Cu at (126.5, 136.6)
- added JP1111: POWER_DOWN, Jumper:SolderJumper-3_P1.3mm_Open_RoundedPad1.0x1.5mm, B.Cu at (131.8, 116.1)
- added JP1112: AN0, Jumper:SolderJumper-3_P1.3mm_Open_RoundedPad1.0x1.5mm, B.Cu at (126.5, 133.8)
- added JP1113: AN1, Jumper:SolderJumper-3_P1.3mm_Open_RoundedPad1.0x1.5mm, B.Cu at (121.3, 136.6)
- added JP1114: AN_EN, Jumper:SolderJumper-3_P1.3mm_Open_RoundedPad1.0x1.5mm, B.Cu at (116.2, 136.6)
- added JP801: SNI_MODE, Jumper:SolderJumper-3_P1.3mm_Open_RoundedPad1.0x1.5mm, F.Cu at (132.7, -17.3)
- added JP802: PHY_AD1, Jumper:SolderJumper-3_P1.3mm_Open_RoundedPad1.0x1.5mm, F.Cu at (132.7, -21.2)
- added JP803: PHY_AD2, Jumper:SolderJumper-3_P1.3mm_Open_RoundedPad1.0x1.5mm, F.Cu at (149.7, -17.3)
- added JP804: PHY_AD3, Jumper:SolderJumper-3_P1.3mm_Open_RoundedPad1.0x1.5mm, F.Cu at (144.0, -13.5)
- added JP805: PHY_AD4, Jumper:SolderJumper-3_P1.3mm_Open_RoundedPad1.0x1.5mm, F.Cu at (138.4, -9.67)
- added JP806: MDIX_EN, Jumper:SolderJumper-3_P1.3mm_Open_RoundedPad1.0x1.5mm, F.Cu at (149.7, -21.2)
- added JP807: MII_MODE, Jumper:SolderJumper-3_P1.3mm_Open_RoundedPad1.0x1.5mm, F.Cu at (144.0, -17.3)
- added JP808: PHY_AD0, Jumper:SolderJumper-3_P1.3mm_Open_RoundedPad1.0x1.5mm, F.Cu at (144.0, -9.67)
- added JP809: LED_CFG, Jumper:SolderJumper-3_P1.3mm_Open_RoundedPad1.0x1.5mm, F.Cu at (138.4, -13.5)
- added JP810: ~RESET, Jumper:SolderJumper-3_P1.3mm_Open_RoundedPad1.0x1.5mm, F.Cu at (132.7, -9.67)
- added JP811: POWER_DOWN, Jumper:SolderJumper-3_P1.3mm_Open_RoundedPad1.0x1.5mm, F.Cu at (144.0, -21.2)
- added JP812: AN0, Jumper:SolderJumper-3_P1.3mm_Open_RoundedPad1.0x1.5mm, F.Cu at (138.4, -17.3)
- added JP813: AN1, Jumper:SolderJumper-3_P1.3mm_Open_RoundedPad1.0x1.5mm, F.Cu at (132.7, -13.5)
- added JP814: AN_EN, Jumper:SolderJumper-3_P1.3mm_Open_RoundedPad1.0x1.5mm, F.Cu at (138.4, -21.2)
- added JP901: SNI_MODE, Jumper:SolderJumper-3_P1.3mm_Open_RoundedPad1.0x1.5mm, B.Cu at (134.2, 80.3)
- added JP902: PHY_AD1, Jumper:SolderJumper-3_P1.3mm_Open_RoundedPad1.0x1.5mm, B.Cu at (134.5, 86.9)
- added JP903: PHY_AD2, Jumper:SolderJumper-3_P1.3mm_Open_RoundedPad1.0x1.5mm, B.Cu at (131.8, 86.9)
- added JP904: PHY_AD3, Jumper:SolderJumper-3_P1.3mm_Open_RoundedPad1.0x1.5mm, B.Cu at (139.8, 80.3)
- added JP905: PHY_AD4, Jumper:SolderJumper-3_P1.3mm_Open_RoundedPad1.0x1.5mm, B.Cu at (137.0, 80.3)
- added JP906: MDIX_EN, Jumper:SolderJumper-3_P1.3mm_Open_RoundedPad1.0x1.5mm, B.Cu at (137.3, 93.7)
- added JP907: MII_MODE, Jumper:SolderJumper-3_P1.3mm_Open_RoundedPad1.0x1.5mm, B.Cu at (131.8, 93.7)
- added JP908: PHY_AD0, Jumper:SolderJumper-3_P1.3mm_Open_RoundedPad1.0x1.5mm, B.Cu at (137.3, 86.9)
- added JP909: LED_CFG, Jumper:SolderJumper-3_P1.3mm_Open_RoundedPad1.0x1.5mm, B.Cu at (134.5, 93.7)
- added JP910: ~RESET, Jumper:SolderJumper-3_P1.3mm_Open_RoundedPad1.0x1.5mm, B.Cu at (126.0, 100.8)
- added JP911: POWER_DOWN, Jumper:SolderJumper-3_P1.3mm_Open_RoundedPad1.0x1.5mm, B.Cu at (131.4, 80.3)
- added JP912: AN0, Jumper:SolderJumper-3_P1.3mm_Open_RoundedPad1.0x1.5mm, B.Cu at (126.0, 98.0)
- added JP913: AN1, Jumper:SolderJumper-3_P1.3mm_Open_RoundedPad1.0x1.5mm, B.Cu at (120.8, 100.8)
- added JP914: AN_EN, Jumper:SolderJumper-3_P1.3mm_Open_RoundedPad1.0x1.5mm, B.Cu at (115.7, 100.8)
- J1101, J701: moved to B.Cu
- moved C1110 313.7 mm to (122.1, 130.7), turned to 270 degrees
- moved C1111 311.8 mm to (114.4, 127.8), turned to 270 degrees
- moved C1109 307.9 mm to (127.6, 121.4), turned to 0 degrees
- moved D701 304.3 mm to (271.6, 101.1), turned to 90 degrees
- moved U702 301.1 mm to (279.5, 97.1)
- moved TP702 296.4 mm to (286.1, 97.1), turned to 90 degrees
- moved D702 296.1 mm to (271.6, 91.0), turned to 90 degrees
- moved TP703 294.2 mm to (286.1, 86.9), turned to 90 degrees
- moved U703 293.0 mm to (279.5, 86.9)
- moved C706 286.2 mm to (274.1, 100.4), turned to 270 degrees
- moved U705 281.8 mm to (279.5, 75.5)
- moved U701 281.4 mm to (278.3, 38.1)
- moved TP705 281.1 mm to (286.1, 75.5), turned to 90 degrees
- moved U704 280.3 mm to (279.5, 61.8)
- moved C726 279.3 mm to (272.9, 96.6), turned to 90 degrees
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Routing:
- net /PHY3/AN0: track 0.00 -> 68.4 mm, vias 0 -> 1
- net /PHY3/PHY_3V3: track 0.00 -> 62.6 mm, vias 0 -> 28
- net /PHY2/AN0: track 57.1 -> 105.6 mm
- net /PHY3/AN1: track 0.00 -> 46.4 mm, vias 0 -> 1
- net Net-(C1106-Pad2): track 1.79 -> 25.7 mm, vias 0 -> 3
- net GNDD: track 56.4 -> 34.0 mm, vias 67 -> 63
- net /PHY3/PHY_AD3: track 0.00 -> 20.0 mm, vias 0 -> 1
- net /PHY3/RX-: track 0.00 -> 17.1 mm
- net /PHY3/SNI_MODE: track 0.00 -> 17.0 mm, vias 0 -> 1
- net /PHY3/PHY_AD4: track 0.00 -> 16.9 mm, vias 0 -> 1
- net /PHY3/RX+: track 0.00 -> 15.8 mm
- net /PHY3/MDIX_EN: track 0.00 -> 15.6 mm, vias 0 -> 1
- net /PHY3/PHY_AD0: track 0.00 -> 15.3 mm, vias 0 -> 1
- net /PHY3/TD+: track 1.80 -> 16.6 mm
- net /PHY3/TD-: track 2.13 -> 16.5 mm
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- added copper zone on F.Cu, net /PHY3/PHY_3V3
- added copper zone on In2.Cu, net /PHY3/PHY_3V3
Other:
- board size 162.4 x 370.8 mm -> 100 x 100 mm

Commit message: Add files via upload
Parts:
- removed C707, C708, C709, C710: 100u, Capacitor_SMD:C_0603_1608Metric
- removed C719, C720, C721, C722: 10u, Capacitor_SMD:C_0402_1005Metric
- removed C727, C728, C729, C730: 100n, Capacitor_SMD:C_0402_1005Metric
- removed C731: 4u7, Capacitor_SMD:C_0402_1005Metric
- removed C735, C736, C737, C738: 10n, Capacitor_SMD:C_0402_1005Metric
- removed C739, C742: 470n, Capacitor_SMD:C_0402_1005Metric
- removed D702, D703, D704, D705: LED_Small, LED_SMD:LED_0402_1005Metric
- removed the J601 at (11.8, -31.3)
- removed the J602 at (-27.5, -31.3)
- removed J604: Extension Port E, Connector_PinHeader_1.27mm:PinHeader_1x16_P1.27mm_Vertical
- removed J605: Extension Port C, Connector_PinHeader_1.27mm:PinHeader_1x16_P1.27mm_Vertical
- removed JP1001, JP1101, JP801, JP901: SNI_MODE, Jumper:SolderJumper-3_P1.3mm_Open_RoundedPad1.0x1.5mm
- removed JP1002, JP1102, JP802, JP902: PHY_AD1, Jumper:SolderJumper-3_P1.3mm_Open_RoundedPad1.0x1.5mm
- removed JP1003, JP1103, JP803, JP903: PHY_AD2, Jumper:SolderJumper-3_P1.3mm_Open_RoundedPad1.0x1.5mm
- removed JP1004, JP1104, JP804, JP904: PHY_AD3, Jumper:SolderJumper-3_P1.3mm_Open_RoundedPad1.0x1.5mm
- removed JP1005, JP1105, JP805, JP905: PHY_AD4, Jumper:SolderJumper-3_P1.3mm_Open_RoundedPad1.0x1.5mm
- removed JP1006, JP1106, JP806, JP906: MDIX_EN, Jumper:SolderJumper-3_P1.3mm_Open_RoundedPad1.0x1.5mm
- removed JP1007, JP1107, JP807, JP907: MII_MODE, Jumper:SolderJumper-3_P1.3mm_Open_RoundedPad1.0x1.5mm
- removed JP1008, JP1108, JP808, JP908: PHY_AD0, Jumper:SolderJumper-3_P1.3mm_Open_RoundedPad1.0x1.5mm
- removed JP1009, JP1109, JP809, JP909: LED_CFG, Jumper:SolderJumper-3_P1.3mm_Open_RoundedPad1.0x1.5mm
- removed JP1010, JP1110, JP810, JP910: ~RESET, Jumper:SolderJumper-3_P1.3mm_Open_RoundedPad1.0x1.5mm
- removed JP1011, JP1111, JP811, JP911: POWER_DOWN, Jumper:SolderJumper-3_P1.3mm_Open_RoundedPad1.0x1.5mm
- removed JP1012, JP1112, JP812, JP912: AN0, Jumper:SolderJumper-3_P1.3mm_Open_RoundedPad1.0x1.5mm
- removed JP1013, JP1113, JP813, JP913: AN1, Jumper:SolderJumper-3_P1.3mm_Open_RoundedPad1.0x1.5mm
- removed JP1014, JP1114, JP814, JP914: AN_EN, Jumper:SolderJumper-3_P1.3mm_Open_RoundedPad1.0x1.5mm
- removed R1001, R1003, R1005, R1007, R1009, R1012, R1014, R1016, R1025, R1027, R1031, R1036, R1038, R1040, R1101, R1103, R1105, R1107, R1109, R1112, R1114, R1116, R1125, R1127, R1131, R1136, R1138, R1140, R801, R803, R805, R807, R809, R812, R814, R816, R825, R827, R831, R836, R838, R840, R901, R903, R905, R907, R909, R912, R914, R916, R925, R927, R931, R936, R938, R940: 2k2, Resistor_SMD:R_0402_1005Metric
- removed R705, R706, R707, R708: 200, Resistor_SMD:R_0402_1005Metric
- removed R709, R710, R711, R712: 0, Resistor_SMD:R_0402_1005Metric
- removed TP703, TP704, TP705, TP706: TP 3.3V VCCAUX, TestPoint:TestPoint_Keystone_5015_Micro-Minature
- removed U703, U704, U705, U706: AMS1117-3.3, Package_TO_SOT_SMD:SOT-223-3_TabPin2
- added C1012: 100n, Capacitor_SMD:C_0402_1005Metric, F.Cu at (168.2, 78.9)
- added D707: INIT, LED_SMD:LED_0603_1608Metric, F.Cu at (167.3, 100.6)
- added J103: POWER 5V, Connector_PinHeader_2.54mm:PinHeader_1x03_P2.54mm_Vertical, F.Cu at (181.8, 41.2)
- added Q701: 2N3904, Package_TO_SOT_SMD:SOT-23, F.Cu at (169.6, 85.5)
- added R1141: 100, Resistor_SMD:R_0402_1005Metric, F.Cu at (189.5, 67.2)
- added R1142: 100, Resistor_SMD:R_0402_1005Metric, F.Cu at (191.6, 67.2)
- added R1143: 1k, Resistor_SMD:R_0402_1005Metric, F.Cu at (186.4, 77.1)
- added R1144: 1k, Resistor_SMD:R_0402_1005Metric, F.Cu at (185.4, 77.1)
- added R1145: 1k, Resistor_SMD:R_0402_1005Metric, F.Cu at (184.4, 77.1)
- added R1146: 1k, Resistor_SMD:R_0402_1005Metric, F.Cu at (183.3, 77.1)
- added R1147: 2k2, Resistor_SMD:R_0402_1005Metric, F.Cu at (141.2, 99.9)
- added R1148: 2k2, Resistor_SMD:R_0402_1005Metric, F.Cu at (163.0, 77.9)
- added R714: 100, Resistor_SMD:R_0402_1005Metric, F.Cu at (167.3, 75.9)
- added R715: 200, Resistor_SMD:R_0402_1005Metric, F.Cu at (171.5, 88.4)
- added R716: 200, Resistor_SMD:R_0402_1005Metric, F.Cu at (179.4, 79.4)
- added R717: 100, Resistor_SMD:R_0402_1005Metric, F.Cu at (168.6, 76.9)
- added R718: 10k, Resistor_SMD:R_0402_1005Metric, F.Cu at (168.7, 83.2)
- added R719: 2k2, Resistor_SMD:R_0402_1005Metric, F.Cu at (168.7, 82.2)
- added R720: 200, Resistor_SMD:R_0402_1005Metric, F.Cu at (168.7, 101.9)
- added R721: 2k2, Resistor_SMD:R_0402_1005Metric, F.Cu at (166.8, 83.9)
- added R722: 2k2, Resistor_SMD:R_0402_1005Metric, F.Cu at (166.7, 88.3)
- added R723: 2k2, Resistor_SMD:R_0402_1005Metric, F.Cu at (165.1, 102.5)
- added REF**: MountingHole_4.3mm_M4_Pad_Via, MountingHole:MountingHole_4.3mm_M4_Pad_Via, F.Cu at (170.8, 47.8)
- added REF**: MountingHole_4.3mm_M4_Pad_Via, MountingHole:MountingHole_4.3mm_M4_Pad_Via, F.Cu at (207.0, 144.0)
- added REF**: MountingHole_4.3mm_M4_Pad_Via, MountingHole:MountingHole_4.3mm_M4_Pad_Via, F.Cu at (99.0, 144.0)
- added REF**: MountingHole_4.3mm_M4_Pad_Via, MountingHole:MountingHole_4.3mm_M4_Pad_Via, F.Cu at (99.0, 39.0)
- added U708: W25Q128JVS, Package_SO:SOIC-8_5.23x5.23mm_P1.27mm, F.Cu at (173.9, 77.0)
- C1001, C1002, C1008, C1101, C1102, C1108, C801, C802, C808, C901, C902, C908: footprint Capacitor_SMD:C_0603_1608Metric -> Capacitor_SMD:C_0402_1005Metric
- C701, C702, C704, C723, C732, C741, C743: value 4u7 -> 100n
- C703, C711, C716, C724, C740, C746, C747, C748: value 470n -> 100n
- C705, C706: value 100u -> 4u7; footprint Capacitor_SMD:C_0603_1608Metric -> Capacitor_SMD:C_0402_1005Metric
- C712, C713, C714, C715, C744, C745: value 4u7 -> 100n; footprint Capacitor_SMD:C_0603_1608Metric -> Capacitor_SMD:C_0402_1005Metric
- C725: value 1u -> 4u7
- C726: value 100n -> 4u7
- C733: value 100n -> 470n
- C734: value 10n -> 470n
- D1001, D1002, D1003, D1101, D1102, D1103, D301, D302, D303, D304, D305, D306, D307, D401, D402, D403, D404, D405, D406, D407, D601, D602, D603, D604, D605, D701, D801, D802, D803, D901, D902, D903: footprint LED_SMD:LED_0402_1005Metric -> LED_SMD:LED_0603_1608Metric
- D706: value DONE -> INIT; footprint LED_SMD:LED_0402_1005Metric -> LED_SMD:LED_0603_1608Metric
- J101: value Conn_01x10 -> Conn_01x06; footprint Connector_PinHeader_1.00mm:PinHeader_1x10_P1.00mm_Vertical -> Connector_PinHeader_2.54mm:PinHeader_1x06_P2.54mm_Vertical
- J601: renamed from J607; footprint Connector_PinHeader_1.27mm:PinHeader_1x03_P1.27mm_Vertical -> Connector_PinHeader_2.54mm:PinHeader_1x03_P2.54mm_Vertical
- J602: renamed from J608; footprint Connector_PinHeader_1.27mm:PinHeader_1x03_P1.27mm_Vertical -> Connector_PinHeader_2.54mm:PinHeader_1x03_P2.54mm_Vertical
- J603: value Extension Port B -> Debug Header; footprint Connector_PinHeader_1.27mm:PinHeader_1x16_P1.27mm_Vertical -> Connector_PinHeader_2.54mm:PinHeader_2x05_P2.54mm_Vertical
- J606: value Extension Port D -> Exension Port D; footprint Connector_PinHeader_1.27mm:PinHeader_1x16_P1.27mm_Vertical -> Connector_PinHeader_2.54mm:PinHeader_1x08_P2.54mm_Vertical
- J701: footprint Connector_PinHeader_1.27mm:PinHeader_2x07_P1.27mm_Vertical -> Connector_PinHeader_2.54mm:PinHeader_2x07_P2.54mm_Vertical; moved to F.Cu
- J801: moved to B.Cu
- Q201, Q202: footprint Package_TO_SOT_THT:TO-92_Inline -> Package_TO_SOT_SMD:SOT-23
- Y501: footprint Crystal:Crystal_SMD_0603-2Pin_6.0x3.5mm_HandSoldering -> Crystal:Crystal_SMD_0603-2Pin_6.0x3.5mm
- moved J606 247.9 mm to (174.5, 118.3), turned to 90 degrees
- moved D605 247.4 mm to (206.5, 91.7), turned to 180 degrees
- moved SW601 245.7 mm to (206.8, 87.0), turned to 180 degrees
- moved D603 245.1 mm to (206.5, 93.3), turned to 180 degrees
- moved J603 245.1 mm to (187.5, 112.8), turned to 180 degrees
- moved Y601 243.8 mm to (196.9, 90.1), turned to 180 degrees
- moved D601 242.7 mm to (204.4, 105.2)
- moved D602 240.8 mm to (206.5, 94.8), turned to 180 degrees
- moved J601 239.2 mm to (193.5, 109.6), turned to 90 degrees
- moved R601 238.5 mm to (201.4, 109.6), turned to 180 degrees
- moved D604 237.0 mm to (206.5, 90.2), turned to 180 degrees
- moved R605 233.7 mm to (205.2, 103.3), turned to 270 degrees
- moved R603 232.1 mm to (201.4, 113.3), turned to 180 degrees
- moved U601 231.1 mm to (197.7, 102.8), turned to 180 degrees
- moved R610 229.2 mm to (209.2, 91.7), turned to 180 degrees
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Connections:
- net Net-(J701-Pad10) renamed /FPGA/TDI
- net Net-(J701-Pad4) renamed /FPGA/TMS
- net Net-(J701-Pad6) renamed /FPGA/TCK
- net Net-(J701-Pad8) renamed /FPGA/TDO
- C701 pad 1: /FPGA/VCCO_BANK0_3V3 -> /FPGA/VCCO_3V3
- C702 pad 1: /FPGA/VCCAUX_3V3 -> /FPGA/VCCO_3V3
- C703 pad 1: /FPGA/VCCO_BANK0_3V3 -> /FPGA/VCCO_3V3
- C704 pad 1: /FPGA/VCCAUX_3V3 -> /FPGA/VCCO_3V3
- C711 pad 1: /FPGA/VCCO_BANK0_3V3 -> /FPGA/VCCO_3V3
- C712 pad 1: /FPGA/VCCAUX_3V3 -> /FPGA/VCCO_3V3
- C713 pad 1: /FPGA/VCCAUX_3V3 -> /FPGA/VCCO_3V3
- C714 pad 1: /FPGA/VCCO_BANK1_3V3 -> /FPGA/VCCO_3V3
- C715 pad 1: /FPGA/VCCAUX_3V3 -> /FPGA/VCCO_3V3
- C716 pad 1: /FPGA/VCCO_BANK1_3V3 -> /FPGA/VCCO_3V3
- C723 pad 1: /FPGA/VCCAUX_3V3 -> /FPGA/VCCINT_1V2
- C724 pad 1: /FPGA/VCCO_BANK1_3V3 -> /FPGA/VCCO_3V3
- C732 pad 1: /FPGA/VCCO_BANK2_3V3 -> /FPGA/VCCO_3V3
- C740 pad 1: /FPGA/VCCO_BANK2_3V3 -> /FPGA/VCCO_3V3
- C744 pad 1: /FPGA/VCCO_BANK3_3V3 -> /FPGA/VCCO_3V3
- C746 pad 1: /FPGA/VCCO_BANK3_3V3 -> /FPGA/VCCO_3V3
- C748 pad 1: /FPGA/VCCO_BANK3_3V3 -> /FPGA/VCCO_3V3
- D706 pad 2: /FPGA/VCCAUX_3V3 -> Net-(D706-Pad2)
- J101 pad 1: /STM32/SPI1_CS -> /STM32/UART_TX
- J101 pad 2: /STM32/SPI1_SCK -> /STM32/UART_RX
- J101 pad 3: /STM32/SPI1_MISO -> /STM32/ADC1
- J101 pad 4: /STM32/SPI1_MOSI -> /STM32/ADC2
- J101 pad 5: /STM32/UART_TX -> /STM32/I2C_SDA
- J101 pad 6: /STM32/UART_RX -> /STM32/I2C_SCL
- J102 pad 1: +5V -> Net-(J102-Pad1)
- J603 pad 1: Net-(J603-Pad1) -> /STM32/STM_3V3
- J603 pad 10: Net-(J603-Pad10) -> /STM32/NRST
- J603 pad 2: Net-(J603-Pad2) -> /STM32/SYS_JTMS_SWDIO
- J603 pad 3: Net-(J603-Pad3) -> GNDD
- J603 pad 4: Net-(J603-Pad4) -> /STM32/SYS_JTCK_SWCLK
- J603 pad 5: Net-(J603-Pad5) -> GNDD
- J603 pad 6: Net-(J603-Pad6) -> /STM32/SYS_TRACESWO
- J603 pad 9: Net-(J603-Pad9) -> GNDD
- J701 pad 2: /FPGA/VCCAUX_3V3 -> /FPGA/VCCO_3V3
- R1002 pad 1: Net-(JP1001-Pad3) -> /PHY2/SNI_MODE
- R1004 pad 1: Net-(JP1002-Pad3) -> /FPGA/PHY2_RXD_0
- R1006 pad 1: Net-(JP1003-Pad3) -> /FPGA/PHY2_RXD_1
- R1008 pad 1: Net-(JP1004-Pad3) -> /PHY2/PHY_AD3
- R1010 pad 1: Net-(JP1005-Pad3) -> /PHY2/PHY_AD4
- R1011 pad 2: Net-(JP1006-Pad1) -> /PHY2/MDIX_EN
- R1013 pad 2: Net-(JP1007-Pad1) -> /FPGA/PHY2_RX_DV
- R1015 pad 2: Net-(JP1008-Pad1) -> /PHY2/PHY_AD0
- R1024 pad 2: Net-(JP1009-Pad1) -> /PHY2/CRS_DV
- R1026 pad 2: Net-(JP1010-Pad1) -> /FPGA/~PHY2_RESET
- R1030 pad 2: Net-(JP1011-Pad1) -> /FPGA/PHY2_POWER_DOWN
- R1035 pad 2: Net-(JP1012-Pad1) -> /PHY2/AN0
- R1037 pad 2: Net-(JP1013-Pad1) -> /PHY2/AN1
- R1039 pad 2: Net-(JP1014-Pad1) -> /PHY2/AN_EN
- R1102 pad 1: Net-(JP1101-Pad3) -> /PHY3/SNI_MODE
- R1104 pad 1: Net-(JP1102-Pad3) -> /FPGA/PHY3_RXD_0
- R1106 pad 1: Net-(JP1103-Pad3) -> /FPGA/PHY3_RXD_1
- R1108 pad 1: Net-(JP1104-Pad3) -> /PHY3/PHY_AD3
- R1110 pad 1: Net-(JP1105-Pad3) -> /PHY3/PHY_AD4
- R1111 pad 2: Net-(JP1106-Pad1) -> /PHY3/MDIX_EN
- R1113 pad 2: Net-(JP1107-Pad1) -> /FPGA/PHY3_RX_DV
- R1115 pad 2: Net-(JP1108-Pad1) -> /PHY3/PHY_AD0
- R1124 pad 2: Net-(JP1109-Pad1) -> /PHY3/CRS_DV
- R1126 pad 2: Net-(JP1110-Pad1) -> /FPGA/~PHY3_RESET
- R1130 pad 2: Net-(JP1111-Pad1) -> /FPGA/PHY3_POWER_DOWN
- R1135 pad 2: Net-(JP1112-Pad1) -> /PHY3/AN0
- R1137 pad 2: Net-(JP1113-Pad1) -> /PHY3/AN1
- R1139 pad 2: Net-(JP1114-Pad1) -> /PHY3/AN_EN
- R713 pad 1: /FPGA/VCCAUX_3V3 -> /FPGA/VCCO_3V3
- R802 pad 1: Net-(JP801-Pad3) -> /100BASETX-PHY 1/SNI_MODE
- R804 pad 1: Net-(JP802-Pad3) -> /STM32/PHY_RXD_0
- R806 pad 1: Net-(JP803-Pad3) -> /STM32/PHY_RXD_1
- R808 pad 1: Net-(JP804-Pad3) -> /100BASETX-PHY 1/PHY_AD3
- R810 pad 1: Net-(JP805-Pad3) -> /100BASETX-PHY 1/PHY_AD4
- R811 pad 2: Net-(JP806-Pad1) -> /100BASETX-PHY 1/MDIX_EN
- R813 pad 2: Net-(JP807-Pad1) -> /100BASETX-PHY 1/RX_DV
- R815 pad 2: Net-(JP808-Pad1) -> /100BASETX-PHY 1/PHY_AD0
- R824 pad 2: Net-(JP809-Pad1) -> /100BASETX-PHY 1/CRS_DV
- R826 pad 2: Net-(JP810-Pad1) -> /100BASETX-PHY 1/~RESET
- R830 pad 2: Net-(JP811-Pad1) -> /100BASETX-PHY 1/POWER_DOWN
- R835 pad 2: Net-(JP812-Pad1) -> /100BASETX-PHY 1/AN0
- R837 pad 2: Net-(JP813-Pad1) -> /100BASETX-PHY 1/AN1
- R839 pad 2: Net-(JP814-Pad1) -> /100BASETX-PHY 1/AN_EN
- R902 pad 1: Net-(JP901-Pad3) -> /PHY1/SNI_MODE
- R904 pad 1: Net-(JP902-Pad3) -> /FPGA/PHY1_RXD_0
- R906 pad 1: Net-(JP903-Pad3) -> /FPGA/PHY1_RXD_1
- R908 pad 1: Net-(JP904-Pad3) -> /PHY1/PHY_AD3
- R910 pad 1: Net-(JP905-Pad3) -> /PHY1/PHY_AD4
- R911 pad 2: Net-(JP906-Pad1) -> /PHY1/MDIX_EN
- R913 pad 2: Net-(JP907-Pad1) -> /FPGA/PHY1_RX_DV
- R915 pad 2: Net-(JP908-Pad1) -> /PHY1/PHY_AD0
- R924 pad 2: Net-(JP909-Pad1) -> /PHY1/CRS_DV
- R926 pad 2: Net-(JP910-Pad1) -> /FPGA/~PHY1_RESET
- R930 pad 2: Net-(JP911-Pad1) -> /FPGA/PHY1_POWER_DOWN
- R935 pad 2: Net-(JP912-Pad1) -> /PHY1/AN0
- R937 pad 2: Net-(JP913-Pad1) -> /PHY1/AN1
- R939 pad 2: Net-(JP914-Pad1) -> /PHY1/AN_EN
- SW701 pad 1: Net-(SW701-Pad1) -> /STM32/FPGA_PROGRAM
- U1002 pad 34: /FPGA/CLK_OUT -> /PHY2/CLK_X1
- U1102 pad 34: /FPGA/CLK_OUT -> /PHY3/CLK_X1
- U602 pad 35: Net-(J603-Pad1) -> Net-(U602-Pad35)
- U602 pad 36: Net-(J603-Pad2) -> Net-(U602-Pad36)
- U602 pad 47: Net-(J603-Pad11) -> Net-(U602-Pad47)
- U602 pad 53: Net-(J603-Pad15) -> Net-(U602-Pad53)
- U602 pad 54: Net-(J603-Pad16) -> Net-(U602-Pad54)
- U602 pad 58: Net-(J606-Pad12) -> Net-(U602-Pad58)
- U602 pad 59: Net-(J606-Pad13) -> Net-(U602-Pad59)
- U602 pad 60: Net-(J606-Pad14) -> Net-(U602-Pad60)
- U602 pad 61: Net-(J606-Pad15) -> Net-(U602-Pad61)
- U602 pad 62: Net-(J606-Pad16) -> Net-(U602-Pad62)
- U602 pad 68: Net-(J602-Pad10) -> /STM32/FPGA_INIT
- U602 pad 69: Net-(J602-Pad11) -> /STM32/FPGA_PROGRAM
- U602 pad 70: Net-(J602-Pad12) -> /FPGA/DONE
- U602 pad 90: Net-(J603-Pad5) -> Net-(U602-Pad90)
- U602 pad 91: Net-(J603-Pad6) -> Net-(U602-Pad91)
- U602 pad 95: Net-(J603-Pad9) -> Net-(U602-Pad95)
- U602 pad 96: Net-(J603-Pad10) -> Net-(U602-Pad96)
- U707 pad 1: Net-(U707-Pad1) -> /FPGA/PHY1_POWER_DOWN
- U707 pad 10: Net-(U707-Pad10) -> /FPGA/PHY1_RXD_0
- U707 pad 100: /FPGA/PHY3_RXD_1 -> /PHY3/CLK_X1
- U707 pad 101: /FPGA/PHY3_RXD_0 -> Net-(U707-Pad101)
- U707 pad 102: /FPGA/PHY3_TX_EN -> Net-(U707-Pad102)
- U707 pad 103: /FPGA/VCCO_BANK1_3V3 -> /FPGA/VCCO_3V3
- U707 pad 104: /FPGA/PHY3_TXD_1 -> Net-(U707-Pad104)
- U707 pad 105: /FPGA/PHY3_TXD_0 -> /FPGA/~PHY3_RESET
- U707 pad 111: /USB-UART/UART-TX -> /FPGA/PHY2_POWER_DOWN
- U707 pad 112: /USB-UART/UART-RX -> /FPGA/PHY2_TXD_1
- U707 pad 114: /FPGA/PHY1_POWER_DOWN -> /FPGA/PHY2_TXD_0
- U707 pad 115: /FPGA/~PHY1_RESET -> /FPGA/PHY2_TX_EN
- U707 pad 116: /PHY1/MDIO -> /FPGA/PHY2_RXD_1
- U707 pad 117: /PHY1/MDC -> /FPGA/PHY2_RXD_0
- U707 pad 118: /PHY1/CRS_DV -> /PHY2/CRS_DV
- U707 pad 119: /FPGA/PHY1_RX_DV -> /FPGA/PHY2_RX_DV
- U707 pad 120: /FPGA/PHY1_RXD_1 -> /PHY2/CLK_X1
- U707 pad 121: /FPGA/PHY1_RXD_0 -> Net-(U707-Pad121)
- U707 pad 122: /FPGA/VCCO_BANK0_3V3 -> /FPGA/VCCO_3V3
- U707 pad 123: /FPGA/PHY1_TX_EN -> Net-(U707-Pad123)
- U707 pad 124: /FPGA/PHY1_TXD_1 -> Net-(U707-Pad124)
- U707 pad 125: /FPGA/VCCO_BANK0_3V3 -> /FPGA/VCCO_3V3
- U707 pad 126: /FPGA/PHY1_TXD_0 -> Net-(U707-Pad126)
- U707 pad 127: /PHY1/CLK_OUT -> /PHY2/CLK_OUT
- U707 pad 129: /FPGA/VCCAUX_3V3 -> /FPGA/VCCO_3V3
- U707 pad 131: /PHY2/CLK_OUT -> Net-(U707-Pad131)
- U707 pad 132: /FPGA/PHY2_POWER_DOWN -> /FPGA/~PHY2_RESET
- U707 pad 133: /FPGA/~PHY2_RESET -> /PHY2/MDIO
- U707 pad 134: /PHY2/MDIO -> /PHY2/MDC
- U707 pad 135: /FPGA/VCCO_BANK0_3V3 -> /FPGA/VCCO_3V3
- U707 pad 137: /PHY2/MDC -> Net-(U707-Pad137)
- U707 pad 138: /PHY2/CRS_DV -> Net-(U707-Pad138)
- U707 pad 139: /FPGA/PHY2_RX_DV -> Net-(U707-Pad139)
- U707 pad 140: /FPGA/PHY2_RXD_1 -> Net-(U707-Pad140)
- U707 pad 141: /FPGA/PHY2_RXD_0 -> Net-(U707-Pad141)
- U707 pad 142: /FPGA/PHY2_TX_EN -> Net-(U707-Pad142)
- U707 pad 143: /FPGA/PHY2_TXD_1 -> Net-(U707-Pad143)
- U707 pad 144: /FPGA/PHY2_TXD_0 -> Net-(R1147-Pad1)
- U707 pad 18: /FPGA/VCCO_BANK3_3V3 -> /FPGA/VCCO_3V3
- U707 pad 20: /FPGA/VCCAUX_3V3 -> /FPGA/VCCO_3V3
- U707 pad 24: Net-(U707-Pad24) -> /PHY1/CLK_OUT
- U707 pad 26: Net-(U707-Pad26) -> /PHY1/MDIO
- U707 pad 27: Net-(U707-Pad27) -> /PHY1/MDC
- U707 pad 31: /FPGA/VCCO_BANK3_3V3 -> /FPGA/VCCO_3V3
- U707 pad 32: Net-(U707-Pad32) -> /PHY1/CRS_DV
- U707 pad 33: Net-(U707-Pad33) -> /FPGA/PHY1_RX_DV
- U707 pad 34: Net-(U707-Pad34) -> /PHY1/CLK_X1
- U707 pad 35: Net-(U707-Pad35) -> /FPGA/~PHY1_RESET
- U707 pad 36: /FPGA/VCCAUX_3V3 -> /FPGA/VCCO_3V3
- U707 pad 37: Net-(SW701-Pad1) -> /STM32/FPGA_PROGRAM
- U707 pad 38: /7seg-display/7SEG-2 -> /FPGA/CSO_B
- U707 pad 39: /7seg-display/7SEG-1 -> /STM32/FPGA_INIT
- U707 pad 4: /FPGA/VCCO_BANK3_3V3 -> /FPGA/VCCO_3V3
- U707 pad 42: /FPGA/VCCO_BANK2_3V3 -> /FPGA/VCCO_3V3
- U707 pad 48: Net-(U707-Pad48) -> /7seg-display/7SEG-1
- U707 pad 50: Net-(U707-Pad50) -> /7seg-display/7SEG-2
- U707 pad 53: /FPGA/VCCAUX_3V3 -> /FPGA/VCCO_3V3
- U707 pad 6: Net-(U707-Pad6) -> /FPGA/PHY1_TXD_1
- U707 pad 60: Net-(U707-Pad60) -> /FPGA/M1
- U707 pad 61: Net-(U707-Pad61) -> /USB-UART/UART-TX
- U707 pad 62: Net-(U707-Pad62) -> /USB-UART/UART-RX
- U707 pad 63: /FPGA/VCCO_BANK2_3V3 -> /FPGA/VCCO_3V3
- U707 pad 64: Net-(U707-Pad64) -> /FPGA/MOSI
- U707 pad 65: Net-(U707-Pad65) -> /FPGA/DIN
- U707 pad 69: Net-(U707-Pad69) -> /FPGA/M0
- U707 pad 7: Net-(U707-Pad7) -> /FPGA/PHY1_TXD_0
- U707 pad 70: /FPGA/CLK_OUT -> /FPGA/CCLK
- U707 pad 71: Net-(D706-Pad1) -> /FPGA/DONE
- U707 pad 73: GNDD -> Net-(R1148-Pad2)
- U707 pad 74: Net-(U707-Pad74) -> /FPGA/PHY3_POWER_DOWN
- U707 pad 76: /FPGA/VCCO_BANK1_3V3 -> /FPGA/VCCO_3V3
- U707 pad 78: Net-(U707-Pad78) -> /FPGA/PHY3_TXD_1
- U707 pad 79: Net-(U707-Pad79) -> /FPGA/PHY3_TXD_0
- U707 pad 8: Net-(U707-Pad8) -> /FPGA/PHY1_TX_EN
- U707 pad 80: Net-(U707-Pad80) -> /FPGA/PHY3_TX_EN
- U707 pad 81: Net-(U707-Pad81) -> /FPGA/PHY3_RXD_1
- U707 pad 82: Net-(U707-Pad82) -> /FPGA/PHY3_RXD_0
- U707 pad 86: /FPGA/VCCO_BANK1_3V3 -> /FPGA/VCCO_3V3
- U707 pad 87: Net-(U707-Pad87) -> /PHY3/CLK_OUT
- U707 pad 9: Net-(U707-Pad9) -> /FPGA/PHY1_RXD_1
- U707 pad 90: /FPGA/VCCAUX_3V3 -> /FPGA/VCCO_3V3
- U707 pad 92: /PHY3/CLK_OUT -> /PHY3/MDIO
- U707 pad 93: /FPGA/PHY3_POWER_DOWN -> Net-(U707-Pad93)
- U707 pad 94: /FPGA/~PHY3_RESET -> /PHY3/MDC
- U707 pad 95: /PHY3/MDIO -> Net-(U707-Pad95)
- U707 pad 97: /PHY3/MDC -> Net-(U707-Pad97)
- U902 pad 34: /FPGA/CLK_OUT -> /PHY1/CLK_X1
Routing:
- net /FPGA/VCCO_3V3: track 0.00 -> 143.0 mm, vias 0 -> 44
- net /FPGA/VCCINT_1V2: track 0.00 -> 80.6 mm, vias 0 -> 5
- net +5V: track 7.88 -> 75.9 mm, vias 0 -> 29
- net /100BASETX-PHY 1/PHY_3V3: track 0.00 -> 62.3 mm, vias 0 -> 20
- net Net-(R1143-Pad1): track 0.00 -> 59.7 mm, vias 0 -> 2
- net Net-(R1144-Pad1): track 0.00 -> 57.0 mm, vias 0 -> 2
- net Net-(R1145-Pad1): track 0.00 -> 55.7 mm, vias 0 -> 2
- net /PHY2/AN0: track 105.6 -> 49.9 mm
- net GNDD: track 34.0 -> 88.9 mm, vias 63 -> 325
- net Net-(R1146-Pad1): track 0.00 -> 53.5 mm, vias 0 -> 2
- net /STM32/ADC2: track 0.00 -> 52.9 mm, vias 0 -> 3
- net /7seg-display/7SEG-2: track 0.00 -> 52.4 mm
- net /7seg-display/7SEG-1: track 0.00 -> 51.2 mm
- net /7seg-display/Digit 2/AK: track 0.00 -> 50.8 mm, vias 0 -> 2
- net /STM32/ADC1: track 0.00 -> 50.5 mm
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- added copper zone on In2.Cu, net +5V
- added copper zone on F.Cu, net /100BASETX-PHY 1/PHY_3V3
- added copper zone on In2.Cu, net /100BASETX-PHY 1/PHY_3V3
- added copper zone on In2.Cu, net /FPGA/VCCO_3V3
- added copper zone on F.Cu, net /STM32/STM_3V3
- added copper zone on In2.Cu, net /STM32/STM_3V3
- added copper zone on B.Cu, net GNDD
Other:
- board size 100 x 100 mm -> 120 x 117 mm
- rule trace_min: 0.2 -> 0
