File: ethernet-sniffer/ethernet-sniffer.sch (KiCad schematic (older format))
At the start: 2 parts, among them J101 Conn_01x10, J102 USB_B_Micro

Commit message: Add files via upload
Parts:
- removed J101: Conn_01x10, Connector_PinHeader_1.00mm:PinHeader_1x10_P1.00mm_Vertical, symbol Connector_Generic:Conn_01x10
- added J101: Conn_01x06, Connector_PinHeader_2.54mm:PinHeader_1x06_P2.54mm_Vertical, symbol Connector_Generic:Conn_01x06
- added J103: POWER 5V, Connector_PinHeader_2.54mm:PinHeader_1x03_P2.54mm_Vertical, symbol Connector_Generic:Conn_01x03
Connections:
- wire segments 123 -> 114
