File: ethernet-sniffer/stm32.sch (KiCad schematic (older format))
At the start: 44 parts, among them J601 Debug Header, J602 Extension Port A, J603 Extension Port B, J604 Extension Port E, J605 Extension Port C, J606 Extension Port D, J607 BOOT0, J608 BOOT1, SW601 SW_Push, U601 AMS1117-3.3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

Commit message: Add files via upload
Parts:
- removed J602: Extension Port A, Connector_PinHeader_1.27mm:PinHeader_1x16_P1.27mm_Vertical, symbol Connector_Generic:Conn_01x16
- removed J603: Extension Port B, Connector_PinHeader_1.27mm:PinHeader_1x16_P1.27mm_Vertical, symbol Connector_Generic:Conn_01x16
- removed J604: Extension Port E, Connector_PinHeader_1.27mm:PinHeader_1x16_P1.27mm_Vertical, symbol Connector_Generic:Conn_01x16
- removed J605: Extension Port C, Connector_PinHeader_1.27mm:PinHeader_1x16_P1.27mm_Vertical, symbol Connector_Generic:Conn_01x16
- removed J606: Extension Port D, Connector_PinHeader_1.27mm:PinHeader_1x16_P1.27mm_Vertical, symbol Connector_Generic:Conn_01x16
- added J606: Exension Port D, Connector_PinHeader_2.54mm:PinHeader_1x08_P2.54mm_Vertical, symbol Connector_Generic:Conn_01x08
- D601, D602, D603, D604, D605: footprint LED_SMD:LED_0402_1005Metric -> LED_SMD:LED_0603_1608Metric
- J601: renamed from J607; footprint Connector_PinHeader_1.27mm:PinHeader_1x03_P1.27mm_Vertical -> Connector_PinHeader_2.54mm:PinHeader_1x03_P2.54mm_Vertical
- J602: renamed from J608; footprint Connector_PinHeader_1.27mm:PinHeader_1x03_P1.27mm_Vertical -> Connector_PinHeader_2.54mm:PinHeader_1x03_P2.54mm_Vertical
- J603: renamed from J601; footprint Connector_PinHeader_1.27mm:PinHeader_2x05_P1.27mm_Vertical -> Connector_PinHeader_2.54mm:PinHeader_2x05_P2.54mm_Vertical
Connections:
- net labels added: FPGA_DONE, FPGA_INIT, FPGA_PROGRAM
- wire segments 224 -> 184
- no-connect marks 25 -> 35
