File: FPGA.sch (KiCad schematic (older format))
At the start: 65 parts, among them J701 JTAG, Q701 2N3904, SW701 RESET, U701 LM317_3PinPackage, U702 AMS1117-3.3, U707 XC6SLX9-TQG144, U708 W25Q128JVS

Commit message: Cleanup
Connections:
- no-connect marks 19 -> 44
Changed lines of the file:
@@
 	1    0    0    -1
 $EndComp
+NoConn ~ 13800 6350
+NoConn ~ 13800 6450
+NoConn ~ 13800 6850
+NoConn ~ 13800 6950
+NoConn ~ 13800 7050
+NoConn ~ 13800 7150
+NoConn ~ 13800 7250
+NoConn ~ 13800 7350
+NoConn ~ 13800 7450
+NoConn ~ 13800 7550
+NoConn ~ 13800 7650
+NoConn ~ 13800 8250
+NoConn ~ 13800 8350
+NoConn ~ 9850 1850
+NoConn ~ 9850 1950
+NoConn ~ 9850 2050
+NoConn ~ 9850 2150
+NoConn ~ 9850 2250
+NoConn ~ 9850 2350
+NoConn ~ 9850 2450
+NoConn ~ 9850 2850
+NoConn ~ 9850 3050
+NoConn ~ 9850 3150
+NoConn ~ 9850 3250
+NoConn ~ 9850 3350
 $EndSCHEMATC
