File: stm32.sch (KiCad schematic (older format))
At the start: 40 parts, among them J601 BOOT0, J602 BOOT1, J603 Debug Header, J606 Exension Port D, SW601 SW_Push, U601 AMS1117-3.3, U602 STM32F107VCTx, Y601 25MHz

Commit message: Cleanup
Connections:
- wire segments 184 -> 176
- no-connect marks 35 -> 43
Changed lines of the file:
@@
 Text Notes 1750 2500 0    50   ~ 0
 I2C
-Wire Wire Line
-	6900 4950 6900 5550
-Wire Wire Line
-	7000 4950 7000 5550
-Wire Wire Line
-	7100 4950 7100 5550
-Wire Wire Line
-	7200 4950 7200 5550
-Wire Wire Line
-	7300 4950 7300 5550
-Wire Wire Line
-	7400 4950 7400 5550
-Wire Wire Line
-	7500 4950 7500 5550
-Wire Wire Line
-	7600 4950 7600 5550
 Text Label 1150 3450 2    50   ~ 0
 ETH_TXD0
@@
 NoConn ~ 8300 4950
 NoConn ~ 8400 4950
+Text HLabel 4650 4050 0    50   UnSpc ~ 0
+STM_3V3
+NoConn ~ 6900 4950
+NoConn ~ 7000 4950
+NoConn ~ 7100 4950
+NoConn ~ 7200 4950
+NoConn ~ 7300 4950
+NoConn ~ 7400 4950
+NoConn ~ 7500 4950
+NoConn ~ 7600 4950
 $EndSCHEMATC

Commit message: PCB layout 90% finished
Parts:
- C601, C604: value 10u -> 1u
- C606: value 1u -> 10n
- Y601: value 25MHz -> X322525MOB4SI 25MHZ; footprint Crystal:Crystal_SMD_5032-4Pin_5.0x3.2mm -> Crystal:Crystal_SMD_3225-4Pin_3.2x2.5mm
- renumbered J606 to J604
Connections:
- net at U602.5 (PE6): now also D602.2 (A)
- net at U602.80 (PC12): no longer D602.2 (A)
Other:
- moved on the sheet: D602
Changed lines of the file:
@@
 $EndComp
 $Comp
-L power:GNDD #PWR0103
+L power:GNDD #PWR0610
 U 1 1 605EFAF6
 P 3450 1200
-F 0 "#PWR0103" H 3450 950 50  0001 C CNN
+F 0 "#PWR0610" H 3450 950 50  0001 C CNN
 F 1 "GNDD" H 3454 1045 50  0000 C CNN
 F 2 "" H 3450 1200 50  0001 C CNN
@@
 P 750 1150
 F 0 "C601" H 842 1196 50  0000 L CNN
-F 1 "10u" H 842 1105 50  0000 L CNN
+F 1 "1u" H 842 1105 50  0000 L CNN
 F 2 "Capacitor_SMD:C_0402_1005Metric" H 750 1150 50  0001 C CNN
 F 3 "~" H 750 1150 50  0001 C CNN
@@
 P 1750 1150
 F 0 "C604" H 1842 1196 50  0000 L CNN
-F 1 "10u" H 1842 1105 50  0000 L CNN
+F 1 "1u" H 1842 1105 50  0000 L CNN
 F 2 "Capacitor_SMD:C_0402_1005Metric" H 1750 1150 50  0001 C CNN
 F 3 "~" H 1750 1150 50  0001 C CNN
@@
 $EndComp
 $Comp
-L power:GNDD #PWR0104
+L power:GNDD #PWR0602
 U 1 1 605FF409
 P 750 1400
-F 0 "#PWR0104" H 750 1150 50  0001 C CNN
+F 0 "#PWR0602" H 750 1150 50  0001 C CNN
 F 1 "GNDD" H 754 1245 50  0000 C CNN
 F 2 "" H 750 1400 50  0001 C CNN
@@
 $EndComp
 $Comp
-L power:+5V #PWR0105
+L power:+5V #PWR0601
 U 1 1 605FF9E5
 P 750 900
-F 0 "#PWR0105" H 750 750 50  0001 C CNN
+F 0 "#PWR0601" H 750 750 50  0001 C CNN
 F 1 "+5V" H 765 1073 50  0000 C CNN
 F 2 "" H 750 900 50  0001 C CNN
@@
 P 2100 1150
 F 0 "C606" H 2192 1196 50  0000 L CNN
-F 1 "1u" H 2192 1105 50  0000 L CNN
+F 1 "10n" H 2192 1105 50  0000 L CNN
 F 2 "Capacitor_SMD:C_0402_1005Metric" H 2100 1150 50  0001 C CNN
 F 3 "~" H 2100 1150 50  0001 C CNN
@@
 $EndComp
 $Comp
-L power:GNDD #PWR0106
+L power:GNDD #PWR0612
 U 1 1 6060CDE4
 P 6200 1200
-F 0 "#PWR0106" H 6200 950 50  0001 C CNN
+F 0 "#PWR0612" H 6200 950 50  0001 C CNN
 F 1 "GNDD" H 6300 1050 50  0000 R CNN
 F 2 "" H 6200 1200 50  0001 C CNN
@@
 	10550 3800 10550 3750
 $Comp
-L power:GNDD #PWR0107
+L power:GNDD #PWR0614
 U 1 1 60617C42
 P 10650 3800
-F 0 "#PWR0107" H 10650 3550 50  0001 C CNN
+F 0 "#PWR0614" H 10650 3550 50  0001 C CNN
 F 1 "GNDD" H 10654 3645 50  0000 C CNN
 F 2 "" H 10650 3800 50  0001 C CNN
@@
 $EndComp
 $Comp
-L power:GNDD #PWR0108
+L power:GNDD #PWR0603
 U 1 1 60630B81
 P 900 7250
-F 0 "#PWR0108" H 900 7000 50  0001 C CNN
+F 0 "#PWR0603" H 900 7000 50  0001 C CNN
 F 1 "GNDD" H 904 7095 50  0000 C CNN
 F 2 "" H 900 7250 50  0001 C CNN
@@
 	1050 5350 950  5350
 $Comp
-L power:GNDD #PWR0109
+L power:GNDD #PWR0604
 U 1 1 60639DC5
 P 1050 5450
-F 0 "#PWR0109" H 1050 5200 50  0001 C CNN
+F 0 "#PWR0604" H 1050 5200 50  0001 C CNN
 F 1 "GNDD" V 1054 5340 50  0000 R CNN
 F 2 "" H 1050 5450 50  0001 C CNN
@@
 VREF+
 $Comp
-L power:GNDD #PWR0110
+L power:GNDD #PWR0606
 U 1 1 6066FEEC
 P 1750 5300
-F 0 "#PWR0110" H 1750 5050 50  0001 C CNN
+F 0 "#PWR0606" H 1750 5050 50  0001 C CNN
 F 1 "GNDD" H 1754 5145 50  0000 C CNN
 F 2 "" H 1750 5300 50  0001 C CNN
@@
 	1750 5300 1900 5300
 $Comp
-L power:GNDD #PWR0111
+L power:GNDD #PWR0605
 U 1 1 606743FD
 P 1600 5550
-F 0 "#PWR0111" H 1600 5300 50  0001 C CNN
+F 0 "#PWR0605" H 1600 5300 50  0001 C CNN
 F 1 "GNDD" H 1604 5395 50  0000 C CNN
 F 2 "" H 1600 5550 50  0001 C CNN
@@
 P 3400 6800
 F 0 "Y601" H 3544 6846 50  0000 L CNN
-F 1 "25MHz" H 3544 6755 50  0000 L CNN
-F 2 "Crystal:Crystal_SMD_5032-4Pin_5.0x3.2mm" H 3400 6800 50  0001 C CNN
+F 1 "X322525MOB4SI 25MHZ" H 3544 6755 50  0000 L CNN
+F 2 "Crystal:Crystal_SMD_3225-4Pin_3.2x2.5mm" H 3400 6800 50  0001 C CNN
 F 3 "~" H 3400 6800 50  0001 C CNN
 	1    3400 6800
@@
 $EndComp
 $Comp
-L power:GNDD #PWR0112
+L power:GNDD #PWR0608
 U 1 1 60684A9E
 P 3400 6650
-F 0 "#PWR0112" H 3400 6400 50  0001 C CNN
+F 0 "#PWR0608" H 3400 6400 50  0001 C CNN
 F 1 "GNDD" H 3404 6495 50  0000 C CNN
 F 2 "" H 3400 6650 50  0001 C CNN
@@
 $EndComp
 $Comp
-L power:GNDD #PWR0113
+L power:GNDD #PWR0609
 U 1 1 60685054
 P 3400 7250
-F 0 "#PWR0113" H 3400 7000 50  0001 C CNN
+F 0 "#PWR0609" H 3400 7000 50  0001 C CNN
 F 1 "GNDD" H 3404 7095 50  0000 C CNN
 F 2 "" H 3400 7250 50  0001 C CNN
@@
 	4850 6950 4850 6850
 $Comp
-L power:GNDD #PWR0114
+L power:GNDD #PWR0611
 U 1 1 606ACFFE
 P 4850 7250
-F 0 "#PWR0114" H 4850 7000 50  0001 C CNN
+F 0 "#PWR0611" H 4850 7000 50  0001 C CNN
 F 1 "GNDD" H 4854 7095 50  0000 C CNN
 F 2 "" H 4850 7250 50  0001 C CNN
@@
 $EndComp
 $Comp
-L power:GNDD #PWR0115
+L power:GNDD #PWR0607
 U 1 1 606D2746
 P 1750 7250
-F 0 "#PWR0115" H 1750 7000 50  0001 C CNN
+F 0 "#PWR0607" H 1750 7000 50  0001 C CNN
 F 1 "GNDD" H 1754 7095 50  0000 C CNN
 F 2 "" H 1750 7250 50  0001 C CNN
@@
 L Device:LED_Small D602
 U 1 1 60F1B347
-P 10500 2400
-F 0 "D602" H 10650 2450 50  0000 C CNN
-F 1 "LED_Small" H 10500 2286 50  0001 C CNN
-F 2 "LED_SMD:LED_0603_1608Metric" V 10500 2400 50  0001 C CNN
-F 3 "~" V 10500 2400 50  0001 C CNN
-	1    10500 2400
-	-1   0    0    1
+P 7500 5650
+F 0 "D602" H 7650 5700 50  0000 C CNN
+F 1 "LED_Small" H 7500 5536 50  0001 C CNN
+F 2 "LED_SMD:LED_0603_1608Metric" V 7500 5650 50  0001 C CNN
+F 3 "~" V 7500 5650 50  0001 C CNN
+	1    7500 5650
+	0    -1   -1   0
 $EndComp
 $Comp
@@
 U 1 1 60F1C2CF
 P 10500 2500
-F 0 "D603" H 10650 2350 50  0000 C CNN
+F 0 "D603" H 10650 2450 50  0000 C CNN
 F 1 "LED_Small" H 10500 2386 50  0001 C CNN
 F 2 "LED_SMD:LED_0603_1608Metric" V 10500 2500 50  0001 C CNN
@@
 L Device:R_Small_US R607
 U 1 1 60F1D27E
-P 10800 2400
-F 0 "R607" V 10595 2400 50  0001 C CNN
-F 1 "200" V 10750 2250 50  0000 C CNN
-F 2 "Resistor_SMD:R_0402_1005Metric" H 10800 2400 50  0001 C CNN
-F 3 "~" H 10800 2400 50  0001 C CNN
-	1    10800 2400
-	0    1    1    0
+P 7500 5950
+F 0 "R607" V 7295 5950 50  0001 C CNN
+F 1 "200" V 7450 5800 50  0000 C CNN
+F 2 "Resistor_SMD:R_0402_1005Metric" H 7500 5950 50  0001 C CNN
+F 3 "~" H 7500 5950 50  0001 C CNN
+	1    7500 5950
+	-1   0    0    1
 $EndComp
 $Comp
@@
 	9900 2500 9900 2950
 Wire Wire Line
-	10400 2400 9800 2400
-Wire Wire Line
-	9800 2400 9800 2950
+	7500 5550 7500 4950
 Wire Wire Line
 	10600 2700 10700 2700
@@
 	10700 2500 10600 2500
 Wire Wire Line
-	10600 2400 10700 2400
-$Comp
-L power:GNDD #PWR0116
+	7500 5750 7500 5850
+$Comp
+L power:GNDD #PWR0615
 U 1 1 60FB9C3A
 P 11000 2550
-F 0 "#PWR0116" H 11000 2300 50  0001 C CNN
+F 0 "#PWR0615" H 11000 2300 50  0001 C CNN
 F 1 "GNDD" H 11004 2395 50  0000 C CNN
 F 2 "" H 11000 2550 50  0001 C CNN
@@
 	11000 2700 11000 2600
 Wire Wire Line
-	11000 2400 10900 2400
+	7500 6150 7500 6050
 Wire Wire Line
 	10900 2700 11000 2700
@@
 Wire Wire Line
 	10900 2500 11000 2500
-Connection ~ 11000 2500
-Wire Wire Line
-	11000 2500 11000 2400
 Wire Wire Line
 	1050 2150 1100 2150
@@
 FPGA_DONE
 $Comp
-L power:PWR_FLAG #FLG0101
+L power:PWR_FLAG #FLG0601
 U 1 1 5FFBC14C
 P 6400 850
-F 0 "#FLG0101" H 6400 925 50  0001 C CNN
+F 0 "#FLG0601" H 6400 925 50  0001 C CNN
 F 1 "PWR_FLAG" H 6400 1023 50  0000 C CNN
 F 2 "" H 6400 850 50  0001 C CNN
@@
 NoConn ~ 9700 4950
 $Comp
-L Connector_Generic:Conn_01x08 J606
+L Connector_Generic:Conn_01x08 J604
 U 1 1 5F44FFF4
 P 8900 5750
-F 0 "J606" V 9000 5800 50  0000 R CNN
+F 0 "J604" V 9000 5800 50  0000 R CNN
 F 1 "Exension Port D" V 9100 6000 50  0000 R CNN
 F 2 "Connector_PinHeader_2.54mm:PinHeader_1x08_P2.54mm_Vertical" H 8900 5750 50  0001 C CNN
@@
 NoConn ~ 7300 4950
 NoConn ~ 7400 4950
-NoConn ~ 7500 4950
+NoConn ~ 9700 2950
 NoConn ~ 7600 4950
+$Comp
+L power:GNDD #PWR0613
+U 1 1 5EF816BD
+P 7500 6150
+F 0 "#PWR0613" H 7500 5900 50  0001 C CNN
+F 1 "GNDD" H 7504 5995 50  0000 C CNN
+F 2 "" H 7500 6150 50  0001 C CNN
+F 3 "" H 7500 6150 50  0001 C CNN
+	1    7500 6150
+	1    0    0    -1
+$EndComp
 $EndSCHEMATC
